File: ac-timer.brd (EAGLE design)
At the start: 84 x 42 mm, 21 parts, among them U1 ATmega328P-PU, Y1 16MHz 18pF

Commit message: Rotate AC input terminal block.
Parts:
- moved J1 6.02 mm to (5.50, 19.0), turned to 180 degrees
Changed lines of the file:
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@@
 <text x="51" y="37.5" size="1.27" layer="21" ratio="16" rot="R90" align="bottom-center">BLK</text>
 <text x="77" y="17.5" size="1.27" layer="21" ratio="16" align="bottom-center">RTC Module</text>
-<text x="6" y="18" size="1.27" layer="21" ratio="16" rot="SR0" align="bottom-center">120VAC</text>
-<text x="0.5" y="13" size="1.27" layer="21" ratio="16" rot="SR270" align="bottom-center">L      N</text>
+<text x="5.5" y="13.5" size="1.27" layer="21" ratio="16" rot="SR0" align="bottom-center">120VAC</text>
+<text x="5.5" y="23.5" size="1.27" layer="21" ratio="16" rot="SR0" align="bottom-center">L      N</text>
 </plain>
 <attributes>
@@
 <attribute name="VALUE" x="21.246" y="39.294" size="0.4064" layer="27" font="vector"/>
 </element>
-<element name="J1" library="_jc" package="OST-TB-2-3.5MM" value="" x="6" y="13" smashed="yes" rot="R270">
-<attribute name="VALUE" x="0.5" y="16" size="1.27" layer="21" ratio="16" rot="R270"/>
+<element name="J1" library="_jc" package="OST-TB-2-3.5MM" value="" x="5.5" y="19" smashed="yes" rot="R180">
+<attribute name="VALUE" x="8.5" y="24.5" size="1.27" layer="21" ratio="16" rot="R180"/>
 </element>
 <element name="R5" library="_jc" package="M0805" value="330" x="47.5" y="28" smashed="yes" rot="R180">

Commit message: Production candidate 01
Parts:
- removed C10, C9: 27pF, _jc:M0805
- removed C11, C12, C13: 100nF, _jc:M0805
- removed D6: 1N4148, _jc:SOD-323F
- removed R5, R6, R7: 330, _jc:M0805
- added A2: RTC module, _jc:RTC79412
- added C1, C3, C6, C7: 100nF, _jc:M0805
- added C2: 10uF, _jc:M0805
- added C4, C5: 27pF, _jc:M0805
- added D1: 1N4148, _jc:SOD-323F
- added R1: 10K, _jc:M0805
- added R2, R3: 330, _jc:M0805
- A1: value RTC module -> IRM-01-5; device _jc:RTC79412 -> _jc:IRM-01
- J1: device _jc:OST-TB-2-3.5MM -> _jc:OST-TB-2-0.20
- R4: value 10K -> 330
- moved A1 60.6 mm to (12.0, 0.50), turned to 0 degrees
- moved R4 17.8 mm to (50.5, 23.5), turned to 180 degrees
- moved J1 4.53 mm to (6.00, 14.5)
- moved LOGO2 4.30 mm to (3.91, 32.8), flipped to the bottom
- moved S1 2.21 mm to (75.3, 38.1), turned to 180 degrees
- moved U1 2.00 mm to (61.3, 18.2)
- moved L1 1.58 mm to (69.4, 11.9)
- moved Y1 1.50 mm to (52.7, 11.8)
- moved C8 1.01 mm to (57.4, 38.9)
- moved LOGO1 0.71 mm to (0.99, 32.8)
- moved JP1 0.06 mm to (48.1, 37.5)
Connections:
- new net N$8: A1.AC/N, J1.P$2
- new net N$9: A1.AC/L, J1.P$1
- net /RESET: now also D1.A, R1.1; no longer D6.A, R4.1
- net GND: now also A1.V-, A2.8, C1.2, C2.2, C3.2, C4.2, C5.2, C6.2, C7.2; no longer A1.8, C10.2, C11.2, C12.2, C13.2, C9.2
- net N$1: now also R4.2; no longer R7.2
- net N$2: now also R3.2; no longer R6.2
- net N$3: now also R2.2; no longer R5.2
- net N$4: now also C5.1; no longer C10.1
- net N$5: now also C6.1; no longer C13.1
- net N$6: now also C4.1; no longer C9.1
- net N$7: now also C7.1; no longer C12.1
- net PD2: now also A2.3; no longer A1.3
- net PD3: now also R2.1; no longer R5.1
- net PD4: now also R3.1; no longer R6.1
- net SCK: now also R4.1; no longer R7.1
- net SCL: now also A2.6; no longer A1.6
- net SDA: now also A2.5; no longer A1.5
- net VCC: now also A1.V+, A2.7, C1.1, C2.1, C3.1, D1.K, R1.2; no longer A1.7, C11.1, D6.K, R4.2
Routing:
- net PC2: track 0.00 -> 44.4 mm
- net PC3: track 0.00 -> 40.8 mm
- net N$1: track 0.00 -> 39.7 mm
- net PD2: track 0.00 -> 36.9 mm
- net N$2: track 0.00 -> 35.1 mm
- net N$3: track 0.00 -> 30.8 mm
- net /RESET: track 0.00 -> 25.2 mm
- net TXD: track 0.00 -> 23.6 mm
- net RST: track 0.00 -> 22.8 mm
- net SCK: track 0.00 -> 21.7 mm
- net SDA: track 0.00 -> 20.9 mm
- net RXD: track 0.00 -> 19.2 mm
- net SCL: track 0.00 -> 18.9 mm
- net N$9: track 0.00 -> 17.2 mm
- net VCC: track 0.00 -> 11.0 mm
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Other:
- board size 84 x 42 mm -> 86 x 42 mm
- board text added: "AC Timer v1.0"
- board text added: "CC BY-SA 4.0 jc 0623"
- board text added: "L N 120 VAC"
- board text added: "RESET"
- board text added: "open source bit.ly/3pciKlK"
- board text removed: "120VAC"
- board text removed: "L N"
