File: ac-timer.sch (EAGLE design)
At the start: 21 parts, among them U1 ATmega328P-PU, Y1 16MHz 18pF

Commit message: Production candidate 01
Parts:
- removed R7: 330, _jc:R-US_M0805
- added A2: RTC module, _jc:RTC79412
- added C1: 100nF, _jc:C-USM0805
- added C2: 10uF, _jc:C-USM0805
- added R1: 10K, _jc:R-US_M0805
- A1: value RTC module -> IRM-01-5; device _jc:RTC79412 -> _jc:IRM-01
- J1: device _jc:OST-TB-23.5MM -> _jc:OST-TB-20.20IN
- R4: value 10K -> 330
- renumbered C10 to C5, C11 to C3, C12 to C7, C13 to C6, C9 to C4, D6 to D1, R5 to R2, R6 to R3
Connections:
- new net N$8: A1.AC/N, J1.2
- new net N$9: A1.AC/L, J1.1
- net /RESET: now also R1.1; no longer R4.1
- net GND: now also A1.V-, A2.GND, C1.2, C2.2; no longer A1.GND
- net N$1: now also R4.2; no longer R7.2
- net PD2: now also A2.MFP; no longer A1.MFP
- net SCK: now also R4.1; no longer R7.1
- net SCL: now also A2.SCL; no longer A1.SCL
- net SDA: now also A2.SDA; no longer A1.SDA
- net VCC: now also A1.V+, A2.VCC, C1.1, C2.1, R1.2; no longer A1.VCC, R4.2
Other:
- moved on the sheet: A1, R4
